File: Prototype Files/KiCad/SidePiece V1/SidePiece V1.kicad_pcb (KiCad board)
At the start: 2 copper layers, 57.4 x 76.2 mm, 10 parts

Commit message: PCB files
Parts:
- added C1: 100nf, Capacitor_SMD:C_0603_1608Metric, F.Cu at (234.4, 74.0)
- added C10: 1uF, Capacitor_SMD:C_0603_1608Metric, F.Cu at (227.3, 79.3)
- added C11: 100nf, Capacitor_SMD:C_0603_1608Metric, F.Cu at (231.1, 73.3)
- added C12: 10uF, Capacitor_SMD:C_0805_2012Metric, F.Cu at (196.8, 59.0)
- added C13: 10uF, Capacitor_SMD:C_0805_2012Metric, F.Cu at (196.8, 55.4)
- added C14: 100nF, Capacitor_SMD:C_0603_1608Metric, F.Cu at (231.1, 75.8)
- added C15: 15pF, Capacitor_SMD:C_0603_1608Metric, F.Cu at (168.9, 84.1)
- added C16: 15pF, Capacitor_SMD:C_0603_1608Metric, F.Cu at (172.2, 81.6)
- added C2: 100nf, Capacitor_SMD:C_0603_1608Metric, F.Cu at (234.4, 76.5)
- added C3: 100nf, Capacitor_SMD:C_0603_1608Metric, F.Cu at (234.4, 79.0)
- added C4: 100nf, Capacitor_SMD:C_0603_1608Metric, F.Cu at (238.3, 83.6)
- added C5: 100nf, Capacitor_SMD:C_0603_1608Metric, F.Cu at (237.7, 73.7)
- added C6: 100nf, Capacitor_SMD:C_0603_1608Metric, F.Cu at (237.7, 76.2)
- added C7: 100nf, Capacitor_SMD:C_0603_1608Metric, F.Cu at (237.7, 78.8)
- added C8: 1uF, Capacitor_SMD:C_0603_1608Metric, F.Cu at (227.3, 74.2)
- added C9: 100nf, Capacitor_SMD:C_0603_1608Metric, F.Cu at (227.3, 76.8)
- added D1: TPD1E10B06, Diode_SMD:D_SOD-523, F.Cu at (231.4, 43.0)
- added D2: TPD1E10B06, Diode_SMD:D_SOD-523, F.Cu at (234.5, 43.0)
- added D3: TPD1E10B06, Diode_SMD:D_SOD-523, F.Cu at (238.5, 43.2)
- added J1: USB_C_Receptacle_USB2.0_16P, Connector_USB:USB_C_Receptacle_GCT_USB4105-xx-A_16P_TopMnt_Horizontal, F.Cu at (164.8, 57.4)
- added R1: 27, Resistor_SMD:R_0603_1608Metric, F.Cu at (164.8, 66.2)
- added R2: 27, Resistor_SMD:R_0603_1608Metric, F.Cu at (166.4, 66.2)
- added R3: 5.1k, Resistor_SMD:R_0603_1608Metric, F.Cu at (242.0, 69.2)
- added R4: 5.1k, Resistor_SMD:R_0603_1608Metric, F.Cu at (242.0, 71.7)
- added R5: DNF, Resistor_SMD:R_0603_1608Metric, F.Cu at (238.7, 64.8)
- added R6: 1k, Capacitor_SMD:C_0603_1608Metric, F.Cu at (238.7, 67.4)
- added R7: 1k, Resistor_SMD:R_0603_1608Metric, F.Cu at (169.5, 79.0)
- added U1: RP2040, Package_DFN_QFN:QFN-56-1EP_7x7mm_P0.4mm_EP3.2x3.2mm, F.Cu at (165.0, 73.0)
- added U2: NCP1117-3.3_SOT223, Package_TO_SOT_SMD:SOT-223-3_TabPin2, F.Cu at (191.0, 57.4)
- added U3: W25Q128JVS, Package_SO:SOIC-8_5.3x5.3mm_P1.27mm, F.Cu at (156.7, 65.4)
- added Y1: ABM8-272-T3, Crystal:Crystal_SMD_3225-4Pin_3.2x2.5mm, F.Cu at (169.2, 81.6)
- K_0, K_1, K_10, K_3, K_4, K_5, K_6, K_7, K_8, K_9: moved to B.Cu
- moved K_1 38.1 mm to (127.0, 63.1), turned to 180 degrees
- moved K_10 38.1 mm to (127.0, 120.2), turned to 180 degrees
- moved K_4 38.1 mm to (127.0, 82.1), turned to 180 degrees
- moved K_5 38.1 mm to (165.1, 101.2), turned to 180 degrees
- moved K_7 38.1 mm to (127.0, 101.2), turned to 180 degrees
- moved K_8 38.1 mm to (165.1, 120.2), turned to 180 degrees
- moved K_0 0.08 mm to (146.1, 63.1), turned to 180 degrees
- moved K_3 0.08 mm to (146.1, 82.1), turned to 180 degrees
- moved K_6 0.08 mm to (146.1, 101.2), turned to 180 degrees
- moved K_9 0.08 mm to (146.1, 120.2), turned to 180 degrees
Routing:
- net +3.3V: track 0.00 -> 33.5 mm, vias 0 -> 4
- net GND: track 0.00 -> 23.7 mm, vias 0 -> 8
- net +1V1: track 0.00 -> 16.9 mm, vias 0 -> 3
- net /XIN: track 0.00 -> 10.7 mm
- net /QSPI_SD2: track 0.00 -> 10.1 mm
- net /USD_D+: track 0.00 -> 7.31 mm
- net /QSPI_SD3: track 0.00 -> 6.84 mm
- net /USD_D-: track 0.00 -> 6.49 mm
- net /QSPI_SCLK: track 0.00 -> 5.76 mm
- net /XOUT: track 0.00 -> 5.63 mm
- net /QSPI_SD0: track 0.00 -> 4.54 mm
- net Net-(C16-Pad2): track 0.00 -> 3.73 mm
- net +5V: track 0.00 -> 3.64 mm
- net Net-(U1-USB_DP): track 0.00 -> 3.11 mm, vias 0 -> 1
- net Net-(U1-USB_DM): track 0.00 -> 2.62 mm, vias 0 -> 1
- added copper zone on F.Cu, net +3.3V
Other:
- copper layers 2 -> 4
- board text added: "KEEP IN MIND THAT THIS IS FACING THE OTHER WAY"

Commit message: PCB Stuff
Parts:
- removed C5: 100nf, Capacitor_SMD:C_0603_1608Metric
- removed K_0, K_1, K_10, K_3, K_4, K_5, K_6, K_7, K_8, K_9: KEYSW, MX_Alps_Hybrid:MX-1U-NoLED
- added D10: D, Diode_SMD:D_0603_1608Metric, F.Cu at (108.3, 101.3)
- added D11: D, Diode_SMD:D_0603_1608Metric, F.Cu at (108.3, 120.4)
- added D12: D, Diode_SMD:D_0603_1608Metric, F.Cu at (116.6, 137.7)
- added D13: D, Diode_SMD:D_0603_1608Metric, F.Cu at (154.2, 121.4)
- added D4: D, Diode_SMD:D_0603_1608Metric, F.Cu at (127.4, 82.3)
- added D5: D, Diode_SMD:D_0603_1608Metric, F.Cu at (127.4, 101.3)
- added D6: D, Diode_SMD:D_0603_1608Metric, F.Cu at (127.4, 120.4)
- added D7: D, Diode_SMD:D_0603_1608Metric, F.Cu at (135.6, 137.7)
- added D8: D, Diode_SMD:D_0603_1608Metric, F.Cu at (108.3, 82.3)
- added D9: D, Diode_SMD:D_0603_1608Metric, F.Cu at (153.9, 102.4)
- added J3: Conn_01x04_Pin, 1_my_custom_libary_pretty:OLED, F.Cu at (140.8, 102.5)
- added MT1: PEC11R-4215F-S0024, 1_my_custom_libary_pretty:XDCR_PEC11R-4215F-S0024, F.Cu at (146.4, 110.9)
- added MT2: PEC11R-4215F-S0024, 1_my_custom_libary_pretty:XDCR_PEC11R-4215F-S0024, F.Cu at (146.4, 129.9)
- added SW1: SWITCH, 1_my_custom_libary_pretty:Kailh_socket_PG1350, B.Cu at (127.4, 72.8)
- added SW2: SWITCH, 1_my_custom_libary_pretty:Kailh_socket_PG1350, B.Cu at (108.3, 72.8)
- added SW3: SWITCH, 1_my_custom_libary_pretty:Kailh_socket_PG1350, B.Cu at (127.4, 91.8)
- added SW4: SWITCH, 1_my_custom_libary_pretty:Kailh_socket_PG1350, B.Cu at (108.3, 91.8)
- added SW5: SWITCH, 1_my_custom_libary_pretty:Kailh_socket_PG1350, B.Cu at (127.4, 110.9)
- added SW6: SWITCH, 1_my_custom_libary_pretty:Kailh_socket_PG1350, B.Cu at (108.3, 110.9)
- added SW7: SWITCH, 1_my_custom_libary_pretty:Kailh_socket_PG1350, B.Cu at (127.4, 129.9)
- added SW8: SWITCH, 1_my_custom_libary_pretty:Kailh_socket_PG1350, B.Cu at (108.3, 129.9)
- added SW9: SW_Push, 1_my_custom_libary_pretty:SW_SPST_PTS810, F.Cu at (137.6, 65.2)
- moved R6 102.6 mm to (137.7, 84.8), turned to 90 degrees
- moved R4 102.3 mm to (139.7, 69.6), turned to -90 degrees
- moved R5 102.1 mm to (137.7, 79.5), turned to -90 degrees
- moved C7 97.4 mm to (141.7, 95.2), turned to 180 degrees
- moved D3 97.1 mm to (146.2, 73.3), turned to 180 degrees
- moved C3 96.1 mm to (139.2, 91.9), turned to 180 degrees
- moved D2 94.5 mm to (145.7, 75.1), turned to 180 degrees
- moved C14 93.5 mm to (137.7, 73.4), turned to -90 degrees
- moved R3 89.3 mm to (152.7, 69.6), turned to -90 degrees
- moved C6 88.5 mm to (149.6, 84.6)
- moved C2 87.4 mm to (147.3, 83.8), turned to 90 degrees
- moved C4 87.2 mm to (151.1, 87.6)
- moved D1 85.8 mm to (150.6, 71.9)
- moved C9 85.4 mm to (142.2, 84.6), turned to 180 degrees
- moved C10 85.4 mm to (142.2, 86.1), turned to 180 degrees
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Connections:
- U1 pad 13: unconnected-(U1-GPIO10-Pad13) -> R1A
- U1 pad 14: unconnected-(U1-GPIO11-Pad14) -> R1B
- U1 pad 15: unconnected-(U1-GPIO12-Pad15) -> R2A
- U1 pad 16: unconnected-(U1-GPIO13-Pad16) -> R2B
- U1 pad 29: unconnected-(U1-GPIO18-Pad29) -> OLED_SDA
- U1 pad 3: unconnected-(U1-GPIO1-Pad3) -> C0
- U1 pad 30: unconnected-(U1-GPIO19-Pad30) -> OLED_SCL
- U1 pad 4: unconnected-(U1-GPIO2-Pad4) -> C1
- U1 pad 5: unconnected-(U1-GPIO3-Pad5) -> R0
- U1 pad 6: unconnected-(U1-GPIO4-Pad6) -> R1
- U1 pad 7: unconnected-(U1-GPIO5-Pad7) -> R2
- U1 pad 8: unconnected-(U1-GPIO6-Pad8) -> R3
- U1 pad 9: unconnected-(U1-GPIO7-Pad9) -> R4
Routing:
- net C1: track 0.00 -> 126.1 mm, vias 0 -> 5
- net C0: track 0.00 -> 83.4 mm, vias 0 -> 3
- net R3: track 0.00 -> 70.5 mm, vias 0 -> 3
- net R4: track 0.00 -> 64.6 mm, vias 0 -> 5
- net R2: track 0.00 -> 55.2 mm, vias 0 -> 3
- net R2B: track 0.00 -> 42.8 mm
- net R1: track 0.00 -> 41.5 mm, vias 0 -> 3
- net R0: track 0.00 -> 40.3 mm, vias 0 -> 3
- net R2A: track 0.00 -> 37.2 mm
- net +3.3V: track 33.5 -> 59.1 mm, vias 4 -> 11
- net R1B: track 0.00 -> 22.3 mm
- net /USB_BOOT: track 0.00 -> 20.3 mm, vias 0 -> 2
- net GND: track 23.7 -> 42.9 mm, vias 8 -> 42
- net /QSPI_SD0: track 4.54 -> 22.7 mm, vias 0 -> 2
- net /QSPI_SS: track 0.00 -> 17.7 mm
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- added copper zone on In2.Cu, net +3.3V
- added copper zone on B.Cu, net GND
- added copper zone on F.Cu, net GND
- added copper zone on In1.Cu, net GND
- added copper zone on In2.Cu, net GND

Commit message: KiCad Files
Parts:
- added R10: 10k, Resistor_SMD:R_0402_1005Metric, F.Cu at (146.3, 98.6)
- added R9: 10k, Resistor_SMD:R_0402_1005Metric, F.Cu at (143.4, 102.4)
- C1, C10, C11, C2, C3, C4, C6, C7, C8, C9: footprint Capacitor_SMD:C_0603_1608Metric -> Capacitor_SMD:C_0402_1005Metric
- moved C6 7.06 mm to (142.8, 86.2), turned to 135 degrees
- moved C9 1.56 mm to (143.5, 85.5), turned to 135 degrees
- moved C2 1.22 mm to (147.8, 85.0), turned to 45 degrees
- moved C8 0.97 mm to (144.2, 84.8), turned to 135 degrees
- moved C10 0.93 mm to (142.0, 87.0), turned to 135 degrees
- moved C4 0.80 mm to (150.4, 87.4), turned to 45 degrees
- moved R7 0.51 mm to (149.9, 95.5)
- moved C3 0.36 mm to (138.9, 91.7)
- moved R5 0.28 mm to (137.4, 79.5)
- moved R6 0.25 mm to (137.4, 84.8)
- moved C7 0.25 mm to (142.0, 95.2)
Routing:
- net GND: track 42.9 -> 66.6 mm, vias 42 -> 47
- net (no net): track 15.6 -> 6.10 mm
- net /XIN: track 17.3 -> 9.88 mm
- net +1V1: track 20.5 -> 13.3 mm, vias 3 -> 4
- net /QSPI_SCLK: track 18.4 -> 22.5 mm
- net R0: track 40.3 -> 43.6 mm
- net /USB_BOOT: track 20.3 -> 22.8 mm
- net OLED_SDA: track 14.4 -> 16.6 mm
- net +3.3V: track 59.1 -> 60.8 mm, vias 11 -> 8
- net /QSPI_SD0: track 22.7 -> 24.3 mm
- net Net-(U1-USB_DP): track 9.52 -> 11.1 mm
- net /QSPI_SD3: track 18.8 -> 17.4 mm
- net Net-(U1-USB_DM): track 9.41 -> 10.5 mm
- net R1B: track 22.3 -> 23.0 mm
- net /QSPI_SS: track 17.7 -> 18.4 mm
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- removed copper zone on F.Cu, net +3.3V
- removed copper zone on In2.Cu, net +3.3V
