File: Prototype Files/KiCad/SidePiece V1/SidePiece V1.kicad_sch (KiCad schematic)
At the start: 1 part

Commit message: PCB files
Parts:
- removed A1: RaspberryPi_Pico, Module:RaspberryPi_Pico_Common_Unspecified, symbol MCU_Module:RaspberryPi_Pico
- added C1, C11, C2, C3, C4, C5, C6, C7, C9: 100nf, Capacitor_SMD:C_0603_1608Metric, symbol Device:C
- added C10, C8: 1uF, Capacitor_SMD:C_0603_1608Metric, symbol Device:C
- added C12, C13: 10uF, Capacitor_SMD:C_0805_2012Metric, symbol Device:C
- added C14: 100nF, Capacitor_SMD:C_0603_1608Metric, symbol Device:C
- added C15, C16: 15pF, Capacitor_SMD:C_0603_1608Metric, symbol Device:C
- added D1, D2, D3: TPD1E10B06, Diode_SMD:D_SOD-523, symbol Diode:ESD9B5.0ST5G
- added J1: USB_C_Receptacle_USB2.0_16P, Connector_USB:USB_C_Receptacle_GCT_USB4105-xx-A_16P_TopMnt_Horizontal, symbol Connector:USB_C_Receptacle_USB2.0_16P
- added J2: Conn_01x02, symbol Connector_Generic:Conn_01x02
- added R1, R2: 27, Resistor_SMD:R_0603_1608Metric, symbol Device:R
- added R3, R4: 5.1k, Resistor_SMD:R_0603_1608Metric, symbol Device:R
- added R5: DNF, Resistor_SMD:R_0603_1608Metric, symbol Device:R
- added R6: 1k, Capacitor_SMD:C_0603_1608Metric, symbol Device:R
- added R7: 1k, Resistor_SMD:R_0603_1608Metric, symbol Device:R
- added U1: RP2040, Package_DFN_QFN:QFN-56-1EP_7x7mm_P0.4mm_EP3.2x3.2mm, symbol MCU_RaspberryPi:RP2040
- added U2: NCP1117-3.3_SOT223, Package_TO_SOT_SMD:SOT-223-3_TabPin2, symbol Regulator_Linear:NCP1117-3.3_SOT223
- added U3: W25Q128JVS, Package_SO:SOIC-8_5.3x5.3mm_P1.27mm, symbol Memory_Flash:W25Q128JVS
- added Y1: ABM8-272-T3, Crystal:Crystal_SMD_3225-4Pin_3.2x2.5mm, symbol Device:Crystal_GND24
Connections:
- new net: C16.2, R7.2, Y1.3
- new net: J1.A5 (CC1), R3.1
- new net: J1.B5 (CC2), R4.1
- new net: R1.2, U1.47 (USB_DP)
- new net: R2.2, U1.46 (USB_DM)
- new net +1V1: C10.1, C11.1, C9.1, U1.23 (DVDD), U1.45 (VREG_VOUT), U1.50 (DVDD)
- new net +3.3V: C1.1, C12.1, C14.1, C2.1, C3.1, C4.1, C5.1, C6.1, C7.1, C8.1, R5.1, U1.1 (IOVDD), U1.10 (IOVDD), U1.22 (IOVDD), U1.33 (IOVDD), U1.42 (IOVDD), U1.43 (ADC_AVDD), U1.44 (VREG_IN), U1.48 (USB_VDD), U1.49 (IOVDD), U2.2 (VO), U3.8 (VCC)
- new net +5V: C13.1, D1.1 (A1), J1.A4 (VBUS), J1.A9 (VBUS), J1.B4 (VBUS), J1.B9 (VBUS), U2.3 (VI)
- new net GND: C1.2, C10.2, C11.2, C12.2, C13.2, C14.2, C15.1, C16.1, C2.2, C3.2, C4.2, C5.2, C6.2, C7.2, C8.2, C9.2, D1.2 (A2), D2.2 (A2), D3.2 (A2), J1.A1 (GND), J1.A12 (GND), J1.B1 (GND), J1.B12 (GND), J1.S1 (SHIELD), J2.1 (Pin_1), R3.2, R4.2, U1.19 (TESTEN), U1.57 (GND), U2.1 (GND), U3.4 (GND), Y1.2, Y1.4
- new net QSPI_SCLK: U1.52 (QSPI_SCLK), U3.6 (CLK)
- new net QSPI_SD0: U1.53 (QSPI_SD0), U3.5 (DI/IO_{0})
- new net QSPI_SD1: U1.55 (QSPI_SD1), U3.2 (DO/IO_{1})
- new net QSPI_SD2: U1.54 (QSPI_SD2), U3.3 (~{WP}/IO_{2})
- new net QSPI_SD3: U1.51 (QSPI_SD3), U3.7 (~{HOLD}/~{RESET}/IO_{3})
- new net QSPI_SS: R5.2, R6.2, U1.56 (QSPI_SS), U3.1 (~{CS})
- new net RUN: U1.26 (RUN)
- new net SWCLK: U1.24 (SWCLK)
- new net SWD: U1.25 (SWD)
- new net USB_BOOT: J2.2 (Pin_2), R6.1
- new net USD_D+: D2.1 (A1), J1.A6 (D+), J1.B6 (D+), R1.1
- new net USD_D-: D3.1 (A1), J1.A7 (D-), J1.B7 (D-), R2.1
- new net XIN: C15.2, U1.20 (XIN), Y1.1
- new net XOUT: R7.1, U1.21 (XOUT)
- no-connect marks 0 -> 32
Other:
- note added: "CRYSTAL"
- note added: "DECOUPLING CAPACITORS"
- note added: "DECOUPLING CAPACITORS - 1v1"
- note added: "DECOUPLING CAPACITORS - 3v3"
- note added: "DOUBLE CHECK POSITIONING"
- note added: "LINEAR REGULATOR"
- note added: "MEMORY"
- note added: "Place 1uF capacitor close to pin 44"
- note added: "Place 1uF capacitor close to pin 45"
- note added: "Replace with switch or button?"
- note added: "USB"

Commit message: PCB Stuff
Parts:
- removed J2: Conn_01x02, symbol Connector_Generic:Conn_01x02
- added D10, D11, D12, D13, D4, D5, D6, D7, D8, D9: D, Diode_SMD:D_0603_1608Metric, symbol Device:D
- added J3: Conn_01x04_Pin, 1_my_custom_libary_pretty:OLED, symbol Connector:Conn_01x04_Pin
- added MT1, MT2: PEC11R-4215F-S0024, 1_my_custom_libary_pretty:XDCR_PEC11R-4215F-S0024, symbol 1_my_custom_symbol_library:PEC11R-4215F-S0024
- added SW1, SW2, SW3, SW4, SW5, SW6, SW7, SW8: SWITCH, 1_my_custom_libary_pretty:Kailh_socket_PG1350, symbol Switch:SW_Omron_B3FS
- added SW9: SW_Push, 1_my_custom_libary_pretty:SW_SPST_PTS810, symbol Switch:SW_Push
Connections:
- net +3.3V: now also J3.2 (Pin_2)
- net GND: now also J3.1 (Pin_1), MT1.COM, MT1.S1 (SHIELD), MT1.S2 (SHIELD), MT2.COM, MT2.S1 (SHIELD), MT2.S2 (SHIELD), SW9.1
- net USB_BOOT: now also SW9.2
- net R1A: now reaches U1.13 (GPIO10)
- net R1A: now also MT1.A
- net R1B: now reaches U1.14 (GPIO11)
- net R1B: now also MT1.B
- net R2A: now reaches U1.15 (GPIO12)
- net R2A: now also MT2.A
- net R2B: now reaches U1.16 (GPIO13)
- net R2B: now also MT2.B
- net OLED_SDA: now reaches U1.29 (GPIO18)
- net OLED_SDA: now also J3.4 (Pin_4)
- net C0: now reaches U1.3 (GPIO1)
- net C0: now also MT1.2, SW1.2, SW3.2, SW5.2, SW7.2
- net OLED_SCL: now reaches U1.30 (GPIO19)
- net OLED_SCL: now also J3.3 (Pin_3)
- net C1: now reaches U1.4 (GPIO2)
- net C1: now also MT2.2, SW2.2, SW4.2, SW6.2, SW8.2
- net R0: now reaches U1.5 (GPIO3)
- net R0: now also D4.1 (K), D8.1 (K)
- net R1: now reaches U1.6 (GPIO4)
- net R1: now also D10.1 (K), D5.1 (K)
- net R2: now reaches U1.7 (GPIO5)
- net R2: now also D11.1 (K), D6.1 (K)
- net R3: now reaches U1.8 (GPIO6)
- net R3: now also D12.1 (K), D7.1 (K)
- net R4: now reaches U1.9 (GPIO7)
- net R4: now also D13.1 (K), D9.1 (K)
- new net: D4.2 (A), SW1.1
- new net: D11.2 (A), SW6.1
- new net: D12.2 (A), SW8.1
- new net: D8.2 (A), SW2.1
- new net: D10.2 (A), SW4.1
- new net: D7.2 (A), SW7.1
- new net: D6.2 (A), SW5.1
- new net: D5.2 (A), SW3.1
- new net R1A_SW: D9.2 (A), MT1.1
- new net R2A_SW: D13.2 (A), MT2.1
- no-connect marks 32 -> 19
Other:
- note added: "ARRAY"
- note added: "OLED DISPLAY"
- note added: "ROTARY ENCODERS"
- note removed: "Replace with switch or button?"
- moved on the sheet: C1, C10, C11, C12, C13, C14, C15, C16, C2, C3, C4, C5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

Commit message: KiCad Files
Parts:
- removed C6: 100nf, Capacitor_SMD:C_0603_1608Metric, symbol Device:C
- added R10, R9: 10k, Resistor_SMD:R_0402_1005Metric, symbol Device:R
- C1, C10, C11, C2, C3, C4, C7, C8, C9: footprint Capacitor_SMD:C_0603_1608Metric -> Capacitor_SMD:C_0402_1005Metric
- C6: renamed from C5; value 100nf -> 220nf; footprint Capacitor_SMD:C_0603_1608Metric -> Capacitor_SMD:C_0402_1005Metric
Connections:
- net +3.3V: now also R10.1, R9.1
- net OLED_SCL: now also R10.2
- net OLED_SDA: now also R9.2
Other:
- moved on the sheet: C1, C2, C3, C4, C6, C7, C8
